File: PSU Schematic.brd (EAGLE design)
At the start: 50.3 x 100 mm, 19 parts, among them IC1 LM34, J1 POWERPOLE_POWER45A, J2 FUSEATC, J3 POWERPOLE_POWER45A, J4 FUSEATC

Commit message: Moar Vias
Routing:
- net GND: vias 71 -> 80
Other:
- outline, holes or cut-outs redrawn
Changed lines of the file:
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@@
 <wire x1="50.3" y1="0" x2="50.3" y2="96.087553125" width="0.4064" layer="20"/>
 <wire x1="50.3" y1="96.087553125" x2="46.387553125" y2="100" width="0.4064" layer="20" curve="90"/>
-<wire x1="46.387553125" y1="100" x2="3.41420625" y2="100" width="0.4064" layer="20"/>
-<wire x1="3.41420625" y1="100" x2="0" y2="96.58579375" width="0.4064" layer="20" curve="90"/>
-<wire x1="0" y1="96.58579375" x2="0" y2="0" width="0.4064" layer="20"/>
+<wire x1="46.387553125" y1="100" x2="4" y2="100" width="0.4064" layer="20"/>
+<wire x1="4" y1="100" x2="0" y2="96" width="0.4064" layer="20" curve="90"/>
+<wire x1="0" y1="96" x2="0" y2="0" width="0.4064" layer="20"/>
 <wire x1="0" y1="0" x2="50.3" y2="0" width="0.4064" layer="20"/>
-<text x="40" y="35" size="1.778" layer="25" align="bottom-right">HP DPS-600
+<text x="41" y="35" size="1.778" layer="25" font="vector" align="bottom-right">HP DPS-600
 Distribution Brd
 </text>
@@
 <vertex x="39" y="88"/>
 </polygon>
-<text x="1" y="73" size="1.778" layer="25" rot="R270">M0YCH
+<text x="5" y="57" size="1.778" layer="25" font="vector" rot="R90">M0YCH
 radio-noise.net</text>
 </plain>
@@
 <via x="13" y="99" extent="1-16" drill="0.6"/>
 <via x="10" y="99" extent="1-16" drill="0.6"/>
+<via x="1" y="87" extent="1-16" drill="0.6"/>
+<via x="1" y="84" extent="1-16" drill="0.6"/>
+<via x="4" y="84" extent="1-16" drill="0.6"/>
+<via x="4" y="87" extent="1-16" drill="0.6"/>
+<via x="7" y="84" extent="1-16" drill="0.6"/>
+<via x="7" y="87" extent="1-16" drill="0.6"/>
+<via x="1" y="81" extent="1-16" drill="0.6"/>
+<via x="46" y="87" extent="1-16" drill="0.6"/>
+<via x="43" y="87" extent="1-16" drill="0.6"/>
 </signal>
 <signal name="PSON">
@@
 <vertex x="22" y="57"/>
 </polygon>
-<via x="21" y="69" extent="1-16" drill="0.6"/>
-<via x="18" y="69" extent="1-16" drill="0.6"/>
 <via x="15" y="69" extent="1-16" drill="0.6"/>
 <via x="12" y="69" extent="1-16" drill="0.6"/>
 <via x="9" y="69" extent="1-16" drill="0.6"/>
+<via x="18" y="72" extent="1-16" drill="0.6"/>
+<via x="21" y="72" extent="1-16" drill="0.6"/>
+<via x="21" y="66" extent="1-16" drill="0.6"/>
+<via x="18" y="66" extent="1-16" drill="0.6"/>
 </signal>
 <signal name="N$4">
@@
 <vertex x="24" y="79"/>
 </polygon>
-<via x="39" y="69" extent="1-16" drill="0.6"/>
-<via x="36" y="69" extent="1-16" drill="0.6"/>
 <via x="33" y="69" extent="1-16" drill="0.6"/>
 <via x="30" y="69" extent="1-16" drill="0.6"/>
 <via x="27" y="69" extent="1-16" drill="0.6"/>
+<via x="36" y="66" extent="1-16" drill="0.6"/>
+<via x="39" y="66" extent="1-16" drill="0.6"/>
+<via x="39" y="72" extent="1-16" drill="0.6"/>
+<via x="36" y="72" extent="1-16" drill="0.6"/>
 </signal>
 <signal name="N$5">

Commit message: Connector Pin adjustment. More vias
Routing:
- net FAN: track 30.0 -> 31.3 mm
- net 5VCC: track 11.0 -> 12.2 mm
- net VCTRL: track 17.0 -> 18.3 mm
- net GND: track 24.8 -> 23.8 mm, vias 80 -> 82
- net CURRENTSHARE: track 28.2 -> 27.6 mm
Changed lines of the file:
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@@
 </text>
 <polygon width="0.4064" layer="30">
-<vertex x="30" y="14"/>
-<vertex x="41" y="14"/>
-<vertex x="41" y="4"/>
+<vertex x="30" y="12"/>
+<vertex x="40" y="12"/>
+<vertex x="40" y="4"/>
 <vertex x="30" y="4"/>
 </polygon>
@@
 <vertex x="10" y="4"/>
 <vertex x="20" y="4"/>
-<vertex x="20" y="14"/>
-<vertex x="9" y="14"/>
-<vertex x="9" y="4"/>
+<vertex x="20" y="12"/>
+<vertex x="10" y="12"/>
 </polygon>
 <polygon width="0.4064" layer="30">
@@
 <via x="46" y="48" extent="1-16" drill="0.6"/>
 <via x="43" y="48" extent="1-16" drill="0.6"/>
-<wire x1="35.5" y1="17" x2="35.5" y2="22" width="0.127" layer="1"/>
-<wire x1="35.5" y1="22" x2="35.27" y2="22" width="0.127" layer="1"/>
-<wire x1="25" y1="35.5" x2="23.5" y2="34" width="0.127" layer="1"/>
-<wire x1="42" y1="35.5" x2="25" y2="35.5" width="0.127" layer="1"/>
-<wire x1="23.5" y1="34" x2="23.365" y2="33.54" width="0.127" layer="1"/>
 <via x="49" y="33" extent="1-16" drill="0.6"/>
 <via x="49" y="39" extent="1-16" drill="0.6"/>
@@
 <via x="46" y="87" extent="1-16" drill="0.6"/>
 <via x="43" y="87" extent="1-16" drill="0.6"/>
+<wire x1="35.25" y1="17" x2="35.25" y2="22" width="0.127" layer="1"/>
+<wire x1="35.25" y1="22" x2="35.27" y2="22" width="0.127" layer="1"/>
+<wire x1="42" y1="33.75" x2="23.5" y2="33.75" width="0.127" layer="1"/>
+<wire x1="23.5" y1="33.75" x2="23.365" y2="33.54" width="0.127" layer="1"/>
+<polygon width="0.4064" layer="16" thermals="no">
+<vertex x="43" y="39"/>
+<vertex x="38" y="39"/>
+<vertex x="38" y="16"/>
+<vertex x="45" y="16"/>
+<vertex x="45" y="32"/>
+</polygon>
+<polygon width="0.4064" layer="1" thermals="no">
+<vertex x="45" y="39"/>
+<vertex x="38" y="39"/>
+<vertex x="38" y="16"/>
+<vertex x="45" y="16"/>
+</polygon>
+<via x="40" y="36" extent="1-16" drill="0.6"/>
+<via x="40" y="30" extent="1-16" drill="0.6"/>
 </signal>
 <signal name="PSON">
@@
 <contactref element="U$2" pad="SIG8"/>
 <contactref element="U$2" pad="SIG10"/>
-<wire x1="25.5" y1="7.5" x2="27.5" y2="5.5" width="0.127" layer="1"/>
-<wire x1="27.5" y1="5.5" x2="27.69" y2="5.08" width="0.127" layer="1"/>
-<wire x1="25.5" y1="7.5" x2="25.15" y2="7.62" width="0.127" layer="1"/>
-<wire x1="25" y1="8" x2="23" y2="10" width="0.127" layer="1"/>
-<wire x1="23" y1="10" x2="22.61" y2="10.16" width="0.127" layer="1"/>
-<wire x1="25" y1="8" x2="25.15" y2="7.62" width="0.127" layer="1"/>
+<wire x1="27.813" y1="3.81" x2="25.3365" y2="6.2865" width="0.127" layer="1"/>
+<wire x1="25.3365" y1="6.2865" x2="25.15" y2="6.35" width="0.127" layer="1"/>
+<wire x1="27.813" y1="3.81" x2="27.69" y2="3.81" width="0.127" layer="1"/>
+<wire x1="25.146" y1="6.2865" x2="22.6695" y2="8.763" width="0.127" layer="1"/>
+<wire x1="22.6695" y1="8.763" x2="22.61" y2="8.89" width="0.127" layer="1"/>
+<wire x1="25.146" y1="6.2865" x2="25.15" y2="6.35" width="0.127" layer="1"/>
 </signal>
 <signal name="5VCC">
 <contactref element="R4" pad="S"/>
 <contactref element="U$2" pad="SIG3"/>
-<wire x1="23" y1="20.5" x2="25" y2="22.5" width="0.127" layer="16"/>
-<wire x1="23" y1="13" x2="23" y2="20.5" width="0.127" layer="16"/>
-<wire x1="25" y1="22.5" x2="25" y2="22.635" width="0.127" layer="16"/>
-<wire x1="23" y1="13" x2="22.61" y2="12.7" width="0.127" layer="16"/>
+<wire x1="24.9555" y1="14.097" x2="24.9555" y2="22.479" width="0.127" layer="16"/>
+<wire x1="22.6695" y1="11.811" x2="24.9555" y2="14.097" width="0.127" layer="16"/>
+<wire x1="22.6695" y1="11.43" x2="22.6695" y2="11.811" width="0.127" layer="16"/>
+<wire x1="24.9555" y1="22.479" x2="25" y2="22.635" width="0.127" layer="16"/>
+<wire x1="22.6695" y1="11.43" x2="22.61" y2="11.43" width="0.127" layer="16"/>
 </signal>
 <signal name="VCTRL">
 <contactref element="R4" pad="A"/>
 <contactref element="U$2" pad="SIG9"/>
-<wire x1="24" y1="19" x2="27.5" y2="22.5" width="0.127" layer="16"/>
-<wire x1="24" y1="9" x2="24" y2="19" width="0.127" layer="16"/>
-<wire x1="23" y1="8" x2="24" y2="9" width="0.127" layer="16"/>
-<wire x1="27.5" y1="22.5" x2="27.54" y2="22.635" width="0.127" layer="16"/>
-<wire x1="23" y1="8" x2="22.61" y2="7.62" width="0.127" layer="16"/>
+<wire x1="27.432" y1="16.002" x2="27.432" y2="22.479" width="0.127" layer="16"/>
+<wire x1="23.8125" y1="12.3825" x2="27.432" y2="16.002" width="0.127" layer="16"/>
+<wire x1="23.8125" y1="7.62" x2="23.8125" y2="12.3825" width="0.127" layer="16"/>
+<wire x1="22.6695" y1="6.477" x2="23.8125" y2="7.62" width="0.127" layer="16"/>
+<wire x1="27.432" y1="22.479" x2="27.54" y2="22.635" width="0.127" layer="16"/>
+<wire x1="22.6695" y1="6.477" x2="22.61" y2="6.35" width="0.127" layer="16"/>
 </signal>
 <signal name="PPV1">
@@
 <via x="4" y="48" extent="1-16" drill="0.6"/>
 <via x="7" y="48" extent="1-16" drill="0.6"/>
-<wire x1="20" y1="28.5" x2="23" y2="28.5" width="0.127" layer="1"/>
-<wire x1="23" y1="28.5" x2="23.365" y2="28.46" width="0.127" layer="1"/>
-<wire x1="31" y1="20.5" x2="32.5" y2="22" width="0.127" layer="1"/>
-<wire x1="20" y1="20.5" x2="31" y2="20.5" width="0.127" layer="1"/>
-<wire x1="32.5" y1="22" x2="32.73" y2="22" width="0.127" layer="1"/>
 <via x="1" y="33" extent="1-16" drill="0.6"/>
 <via x="1" y="39" extent="1-16" drill="0.6"/>
@@
 <via x="36" y="45" extent="1-16" drill="0.6"/>
 <via x="39" y="45" extent="1-16" drill="0.6"/>
+<wire x1="31.25" y1="20.75" x2="32.5" y2="22" width="0.127" layer="1"/>
+<wire x1="20" y1="20.75" x2="31.25" y2="20.75" width="0.127" layer="1"/>
+<wire x1="32.5" y1="22" x2="32.73" y2="22" width="0.127" layer="1"/>
+<wire x1="20" y1="28.5" x2="23.25" y2="28.5" width="0.127" layer="1"/>
+<wire x1="23.25" y1="28.5" x2="23.365" y2="28.46" width="0.127" layer="1"/>
 </signal>
 <signal name="FAN">
@@
 <wire x1="23.5" y1="31" x2="23.365" y2="31" width="0.127" layer="1"/>
 <wire x1="34" y1="24" x2="34" y2="23.905" width="0.127" layer="1"/>
-<wire x1="29" y1="11.5" x2="28" y2="10.5" width="0.127" layer="16"/>
-<wire x1="29" y1="16" x2="29" y2="11.5" width="0.127" layer="16"/>
-<wire x1="34" y1="21" x2="29" y2="16" width="0.127" layer="16"/>
-<wire x1="34" y1="23.905" x2="34" y2="21" width="0.127" layer="16"/>
-<wire x1="28" y1="10.5" x2="27.69" y2="10.16" width="0.127" layer="16"/>
+<wire x1="27.813" y1="9.3345" x2="27.813" y2="8.9535" width="0.127" layer="1"/>
+<wire x1="29.337" y1="10.8585" x2="27.813" y2="9.3345" width="0.127" layer="1"/>
+<wire x1="29.337" y1="17.145" x2="29.337" y2="10.8585" width="0.127" layer="1"/>
+<wire x1="33.909" y1="21.717" x2="29.337" y2="17.145" width="0.127" layer="1"/>
+<wire x1="33.909" y1="23.8125" x2="33.909" y2="21.717" width="0.127" layer="1"/>
+<wire x1="27.813" y1="8.9535" x2="27.69" y2="8.89" width="0.127" layer="1"/>
+<wire x1="33.909" y1="23.8125" x2="34" y2="23.905" width="0.127" layer="1"/>
 </signal>
 <signal name="CURRENTSHARE">
 <contactref element="CS" pad="1"/>
 <contactref element="U$2" pad="SIG11"/>
-<wire x1="29" y1="25.5" x2="31" y2="27.5" width="0.127" layer="16"/>
-<wire x1="29" y1="18" x2="29" y2="25.5" width="0.127" layer="16"/>
-<wire x1="26.5" y1="15.5" x2="29" y2="18" width="0.127" layer="16"/>
-<wire x1="26.5" y1="6.5" x2="26.5" y2="15.5" width="0.127" layer="16"/>
-<wire x1="25.5" y1="5.5" x2="26.5" y2="6.5" width="0.127" layer="16"/>
-<wire x1="31" y1="27.5" x2="34.33" y2="27.53" width="0.127" layer="16"/>
-<wire x1="25.5" y1="5.5" x2="25.15" y2="5.08" width="0.127" layer="16"/>
+<wire x1="34.29" y1="25.7175" x2="34.29" y2="27.432" width="0.127" layer="16"/>
+<wire x1="27.813" y1="19.2405" x2="34.29" y2="25.7175" width="0.127" layer="16"/>
+<wire x1="27.813" y1="13.9065" x2="27.813" y2="19.2405" width="0.127" layer="16"/>
+<wire x1="26.4795" y1="12.573" x2="27.813" y2="13.9065" width="0.127" layer="16"/>
+<wire x1="26.4795" y1="4.953" x2="26.4795" y2="12.573" width="0.127" layer="16"/>
+<wire x1="25.3365" y1="3.81" x2="26.4795" y2="4.953" width="0.127" layer="16"/>
+<wire x1="34.29" y1="27.432" x2="34.33" y2="27.53" width="0.127" layer="16"/>
+<wire x1="25.3365" y1="3.81" x2="25.15" y2="3.81" width="0.127" layer="16"/>
 </signal>
 </signals>
